File: pcb/bigmuff.kicad_pcb (KiCad board)
At the start: 2 copper layers, 46 parts, among them Q1 BC549, Q2 BC549, Q3 BC549, Q4 BC549

Commit message: pcb progress
Parts:
- moved R10 106.2 mm to (85.9, 139.0), turned to 180 degrees
- moved D1 105.4 mm to (71.9, 123.5)
- moved R20 101.4 mm to (121.6, 164.0), turned to 180 degrees
- moved R9 97.2 mm to (84.0, 115.9), turned to -90 degrees
- moved D2 96.3 mm to (79.5, 118.0), turned to 180 degrees
- moved R19 94.1 mm to (121.7, 151.0), turned to 180 degrees
- moved R22 88.3 mm to (133.1, 164.0), turned to 180 degrees
- moved R17 82.3 mm to (117.9, 123.6), turned to 90 degrees
- moved C5 82.3 mm to (89.0, 134.0), turned to 90 degrees
- moved C6 82.2 mm to (78.5, 131.5), turned to 180 degrees
- moved R21 80.8 mm to (133.1, 151.0), turned to 180 degrees
- moved D4 76.9 mm to (98.9, 123.5)
- moved C12 73.4 mm to (114.1, 160.0), turned to 90 degrees
- moved D3 69.0 mm to (106.5, 118.0), turned to 180 degrees
- moved R15 61.9 mm to (111.5, 116.0), turned to -90 degrees
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Routing:
- net Net-(Q3-B): track 13.8 -> 47.4 mm
- net CLIP_OUT: track 0.00 -> 32.1 mm
- net BOOST_OUT: track 28.4 -> 0.00 mm
- net Net-(C3-Pad2): track 27.7 -> 0.00 mm
- net Net-(Q4-B): track 0.00 -> 23.6 mm
- net Net-(R6-Pad1): track 21.7 -> 0.00 mm
- net Net-(D3-A): track 0.00 -> 19.1 mm
- net Net-(D1-K): track 0.00 -> 16.2 mm
- net Net-(D1-A): track 5.08 -> 20.8 mm
- net Net-(Q4-E): track 0.00 -> 14.2 mm
- net Net-(Q1-E): track 17.3 -> 4.92 mm
- net Net-(Q1-C): track 34.7 -> 23.8 mm
- net Net-(Q4-C): track 0.00 -> 6.50 mm
- net Net-(Q3-E): track 0.00 -> 4.99 mm
- net Net-(Q2-B): track 25.4 -> 29.8 mm
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
Commit message: pcb update
Parts:
- moved Q2 37.0 mm to (110.2, 95.0)
- moved R16 37.0 mm to (139.6, 105.0)
- moved R17 37.0 mm to (132.6, 89.6)
- moved C1 37.0 mm to (92.2, 123.4)
- moved C10 37.0 mm to (138.2, 90.0)
- moved C11 37.0 mm to (145.7, 72.5)
- moved C12 37.0 mm to (128.8, 126.0)
- moved C13 37.0 mm to (146.2, 83.0)
- moved C2 37.0 mm to (114.2, 115.9)
- moved C3 37.0 mm to (111.7, 121.4)
- moved C4 37.0 mm to (116.7, 126.4)
- moved C5 37.0 mm to (103.7, 100.0)
- moved C6 37.0 mm to (93.2, 97.5)
- moved C7 37.0 mm to (103.7, 89.5)
- moved C8 37.0 mm to (121.7, 97.5)
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
Commit message: pcb update
Other:
- board outline added: 50.8 x 109.2 mm
Changed lines of the file:
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@@
 		)
+	)
+	(gr_rect
+		(start 175.26 40.64)
+		(end 226.06 149.86)
+		(stroke
+			(width 0.05)
+			(type default)
+		)
+		(fill no)
+		(layer "Edge.Cuts")
 	)
 	(segment

Commit message: update pcb
Parts:
- C1, C6, C8: footprint Capacitor_THT:CP_Radial_Tantal_D4.5mm_P5.00mm -> Capacitor_THT:C_Axial_L5.1mm_D3.1mm_P7.50mm_Horizontal
- C10, C11, C12, C13, C2, C3, C4, C5, C7, C9: footprint Capacitor_THT:C_Disc_D4.3mm_W1.9mm_P5.00mm -> Capacitor_THT:C_Axial_L5.1mm_D3.1mm_P7.50mm_Horizontal
- R1, R10, R11, R12, R13, R14, R15, R16, R17, R18, R19, R2, R20, R21, R22, R3, R4, R5, R6, R7, R8, R9: footprint Resistor_THT:R_Axial_DIN0207_L6.3mm_D2.5mm_P7.62mm_Horizontal -> Resistor_THT:R_Axial_DIN0207_L6.3mm_D2.5mm_P10.16mm_Horizontal
- RV1, RV2, RV3: footprint Potentiometer_THT:Potentiometer_Alpha_RD901F-40-00D_Single_Vertical -> Potentiometer_THT:Potentiometer_Alps_RK09L_Single_Vertical
- moved RV1 72.5 mm to (81.4, 147.2)
- moved RV3 72.1 mm to (137.2, 147.3)
- moved RV2 71.8 mm to (109.3, 147.3)
- moved C13 42.3 mm to (129.5, 121.9), turned to -90 degrees
- moved C7 41.5 mm to (114.4, 129.5), turned to 0 degrees
- moved R2 38.8 mm to (83.8, 94.0)
- moved R12 35.4 mm to (114.4, 124.5), turned to 0 degrees
- moved R6 34.1 mm to (83.8, 124.5)
- moved Q1 32.0 mm to (78.7, 104.1)
- moved R4 31.9 mm to (83.8, 99.1), turned to 180 degrees
- moved C3 31.2 mm to (81.3, 114.3), turned to 180 degrees
- moved R22 31.1 mm to (144.8, 99.1)
- moved C2 29.1 mm to (88.9, 101.6), turned to -90 degrees
- moved R1 28.7 mm to (83.8, 88.9)
- moved C1 27.2 mm to (88.9, 96.4), turned to 90 degrees
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Routing:
- net Net-(D1-A): track 20.8 -> 73.6 mm
- net CLIP_OUT: track 32.1 -> 55.1 mm
- net Net-(Q2-B): track 29.8 -> 46.5 mm
- net Net-(Q4-C): track 6.50 -> 22.0 mm
- net Net-(Q1-B): track 40.0 -> 27.7 mm
- net Net-(Q1-C): track 23.8 -> 33.7 mm, vias 0 -> 1
- net Net-(Q4-B): track 23.6 -> 33.2 mm
- net Net-(Q1-E): track 4.92 -> 12.3 mm
- net Net-(D3-A): track 19.1 -> 13.8 mm
- net Net-(C10-Pad2): track 0.00 -> 5.13 mm
- net Net-(C1-Pad2): track 10.2 -> 5.08 mm
- net Net-(C11-Pad2): track 0.00 -> 5.08 mm
- net Net-(C7-Pad2): track 7.07 -> 9.60 mm
- net Net-(D1-K): track 16.2 -> 13.8 mm
- net Net-(Q3-E): track 4.99 -> 7.18 mm
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Other:
- board size 50.8 x 109.2 mm -> 107.9 x 81.3 mm

Commit message: updated pcb
Parts:
- added C14: 100uF, Capacitor_THT:CP_Radial_D6.3mm_P2.50mm, F.Cu at (192.4, 56.7)
- added C15: 100nF, Capacitor_THT:C_Axial_L5.1mm_D3.1mm_P7.50mm_Horizontal, F.Cu at (200.0, 56.7)
- added D5: LED, LED_THT:LED_D5.0mm, F.Cu at (207.6, 87.2)
- added D6: 1N5817, Diode_THT:D_DO-41_SOD81_P10.16mm_Horizontal, F.Cu at (187.3, 56.7)
- added J1: Jack-DC, Connector_BarrelJack:BarrelJack_Kycon_KLDX-0202-xC_Horizontal, F.Cu at (167.0, 59.3)
- added J2: AudioJack2, Connector_Audio:Jack_6.35mm_Neutrik_NRJ3HF-1_Horizontal, F.Cu at (127.6, 114.8)
- added J3: AudioJack2, Connector_Audio:Jack_6.35mm_Neutrik_NRJ3HF-1_Horizontal, F.Cu at (210.8, 102.9)
- added R23: 4.7k, Resistor_THT:R_Axial_DIN0207_L6.3mm_D2.5mm_P10.16mm_Horizontal, F.Cu at (207.6, 69.4)
- moved R5 85.1 mm to (149.1, 64.4), turned to -90 degrees
- moved R6 67.4 mm to (149.1, 107.5)
- moved R3 67.4 mm to (149.1, 102.6)
- moved RV1 62.6 mm to (141.6, 130.3)
- moved C3 62.5 mm to (141.5, 97.4)
- moved C13 60.9 mm to (189.7, 112.6), turned to 180 degrees
- moved Q1 60.0 mm to (136.4, 87.3)
- moved RV2 57.8 mm to (164.5, 130.3)
- moved C10 57.7 mm to (184.6, 74.4)
- moved C12 57.7 mm to (200.0, 112.6)
- moved R18 57.7 mm to (199.9, 66.9)
- moved Q4 57.6 mm to (194.8, 87.2)
- moved C7 57.6 mm to (169.5, 112.6)
- moved D3 57.6 mm to (169.5, 77.1)
- moved Q2 57.6 mm to (159.4, 92.3)
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Routing:
- net VDD: track 0.00 -> 123.4 mm
- net Net-(C10-Pad2): track 5.13 -> 89.8 mm, vias 0 -> 2
- net Net-(C11-Pad2): track 5.08 -> 72.4 mm
- net TONE_OUT: track 0.00 -> 41.8 mm, vias 0 -> 1
- net Net-(C3-Pad2): track 0.00 -> 38.3 mm
- net BOOST_OUT: track 0.00 -> 29.1 mm, vias 0 -> 1
- net Net-(R6-Pad1): track 0.00 -> 23.8 mm
- net Net-(C13-Pad2): track 0.00 -> 20.0 mm
- net Net-(Q1-C): track 33.7 -> 45.5 mm, vias 1 -> 0
- net Net-(D6-A): track 0.00 -> 11.7 mm
- net CLIP_OUT: track 55.1 -> 64.8 mm
- net Net-(Q4-C): track 22.0 -> 29.6 mm
- net Net-(Q1-E): track 12.3 -> 18.4 mm
- net Net-(D5-A): track 0.00 -> 5.08 mm
- net Net-(Q1-B): track 27.7 -> 25.1 mm
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Other:
- board size 107.9 x 81.3 mm -> 118.5 x 88.9 mm

Commit message: updated pcb
Parts:
- removed J3: AudioJack2, Connector_Audio:Jack_6.35mm_Neutrik_NRJ3HF-1_Horizontal
- added J4: Barrel_Jack_Switch, Connector_BarrelJack:BarrelJack_Kycon_KLDX-0202-xC_Horizontal, F.Cu at (210.5, 63.0)
- added TP1: Input, Connector_PinHeader_1.00mm:PinHeader_1x01_P1.00mm_Vertical, F.Cu at (126.5, 59.0)
- added TP2: Boost, Connector_PinHeader_1.00mm:PinHeader_1x01_P1.00mm_Vertical, F.Cu at (140.5, 59.0)
- added TP3: Clip 1, Connector_PinHeader_1.00mm:PinHeader_1x01_P1.00mm_Vertical, F.Cu at (154.5, 59.0)
- added TP4: Clip 2, Connector_PinHeader_1.00mm:PinHeader_1x01_P1.00mm_Vertical, F.Cu at (168.5, 59.0)
- added TP5: Tone, Connector_PinHeader_1.00mm:PinHeader_1x01_P1.00mm_Vertical, F.Cu at (182.5, 59.0)
- added TP6: Output, Connector_PinHeader_1.00mm:PinHeader_1x01_P1.00mm_Vertical, F.Cu at (196.5, 59.0)
- J1: value Jack-DC -> NRJ4HF; footprint Connector_BarrelJack:BarrelJack_Kycon_KLDX-0202-xC_Horizontal -> Connector_Audio:Jack_6.35mm_Neutrik_NMJ4HFD3_Horizontal
- J2: value AudioJack2 -> NRJ4HF; footprint Connector_Audio:Jack_6.35mm_Neutrik_NRJ3HF-1_Horizontal -> Connector_Audio:Jack_6.35mm_Neutrik_NMJ4HFD3_Horizontal
- moved J2 78.1 mm to (204.2, 99.2), turned to 0 degrees
- moved J1 75.9 mm to (115.9, 115.5), turned to 180 degrees
- moved C14 23.3 mm to (203.2, 77.4), turned to -90 degrees
- moved C15 23.3 mm to (210.8, 77.4), turned to -90 degrees
- moved D6 20.2 mm to (200.0, 72.5), turned to 0 degrees
- moved D5 19.3 mm to (214.0, 69.0), turned to 0 degrees
- moved RV1 12.4 mm to (129.5, 133.1)
- moved R23 11.5 mm to (215.9, 77.4)
- moved D3 8.85 mm to (161.1, 79.9)
- moved Q2 8.85 mm to (151.0, 95.1)
- moved Q4 8.85 mm to (186.4, 90.1)
- moved R14 8.85 mm to (161.1, 100.2)
- moved R5 8.85 mm to (140.7, 67.2)
- moved C7 8.85 mm to (161.1, 115.5)
- moved R12 8.85 mm to (161.1, 110.4)
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Connections:
- J2 pad S: unconnected-(J2-PadS) -> GND
- J2 pad T: unconnected-(J2-PadT) -> OUT
Routing:
- net OUT: track 0.00 -> 86.6 mm, vias 0 -> 2
- net BOOST_OUT: track 29.1 -> 107.6 mm, vias 1 -> 2
- net TONE_OUT: track 41.8 -> 109.3 mm, vias 1 -> 3
- net IN: track 0.00 -> 60.9 mm
- net Net-(C13-Pad2): track 20.0 -> 48.4 mm
- net Net-(D5-A): track 5.08 -> 21.2 mm
- net Net-(D1-A): track 73.6 -> 88.0 mm
- net Net-(C10-Pad2): track 89.8 -> 102.8 mm, vias 2 -> 0
- net CLIP_OUT: track 64.8 -> 77.3 mm
- net Net-(D6-A): track 11.7 -> 21.4 mm
- net VDD: track 123.4 -> 126.8 mm
- net Net-(R6-Pad1): track 23.8 -> 25.9 mm
- net Net-(C11-Pad2): track 72.4 -> 70.3 mm
- net Net-(C3-Pad2): track 38.3 -> 36.8 mm
- net Net-(Q4-C): track 29.6 -> 30.4 mm
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- added copper zone on B.Cu, net GND
- added copper zone on F.Cu, net GND
Other:
- board size 118.5 x 88.9 mm -> 120 x 90 mm
- board text added: "BIG MUFF"
- board text added: "BOOST"
- board text added: "CLIP 1"
- board text added: "CLIP 2"
- board text added: "IN"
- board text added: "IN BOOST"
- board text added: "OUT"
- board text added: "OUT BOOST"
- board text added: "SLEEVE"
- board text added: "TIP"
- board text added: "TONE"
- board text added: "UF AES - FALL 2026"
- board text added: "VOLUME"
- board text added: "π"

Commit message: updated test points
Parts:
- TP1, TP2, TP3, TP4, TP5, TP6: footprint Connector_PinHeader_1.00mm:PinHeader_1x01_P1.00mm_Vertical -> Connector_PinHeader_1.00mm:PinHeader_1x02_P1.00mm_Vertical
- moved R23 10.1 mm to (216.0, 87.5), turned to 90 degrees
- moved C14 1.70 mm to (201.5, 77.4)
- moved D6 1.00 mm to (199.0, 72.5)
- moved LED 0.71 mm to (213.5, 69.5)
- turned TP1 to 180 degrees
- turned TP2 to 180 degrees
- turned TP3 to 180 degrees
- turned TP4 to 180 degrees
- turned TP5 to 180 degrees
- turned TP6 to 180 degrees
- renumbered D5 to LED
Routing:
- net Net-(D5-A): track 21.2 -> 7.86 mm
- net VDD: track 126.8 -> 133.0 mm
- net OUT: track 86.6 -> 92.8 mm
- net Net-(R6-Pad1): track 25.9 -> 25.3 mm
Other:
- board text added: "S"
- board text added: "T"
- board text removed: "SLEEVE"
- board text removed: "TIP"

Commit message: update pcb
Parts:
- removed LED: LED, LED_THT:LED_D5.0mm
- removed TP1: Input, Connector_PinHeader_1.00mm:PinHeader_1x02_P1.00mm_Vertical
- removed TP2: Boost, Connector_PinHeader_1.00mm:PinHeader_1x02_P1.00mm_Vertical
- removed TP3: Clip 1, Connector_PinHeader_1.00mm:PinHeader_1x02_P1.00mm_Vertical
- removed TP4: Clip 2, Connector_PinHeader_1.00mm:PinHeader_1x02_P1.00mm_Vertical
- removed TP5: Tone, Connector_PinHeader_1.00mm:PinHeader_1x02_P1.00mm_Vertical
- removed TP6: Output, Connector_PinHeader_1.00mm:PinHeader_1x02_P1.00mm_Vertical
- added D5: LED, LED_THT:LED_D5.0mm, F.Cu at (215.9, 70.5)
- added G***: LOGO, LOGO, F.Cu at (111.0, 127.5)
- added G***: LOGO, LOGO, F.Cu at (209.5, 127.5)
- added GND: Conn_01x02_Pin, Connector_PinHeader_2.54mm:PinHeader_1x02_P2.54mm_Vertical, F.Cu at (116.5, 57.5)
- added J3: Conn_01x02_Pin, Connector_PinHeader_2.54mm:PinHeader_1x02_P2.54mm_Vertical, F.Cu at (121.0, 57.5)
- added J5: Conn_01x02_Pin, Connector_PinHeader_2.54mm:PinHeader_1x02_P2.54mm_Vertical, F.Cu at (137.5, 57.5)
- added J6: Conn_01x02_Pin, Connector_PinHeader_2.54mm:PinHeader_1x02_P2.54mm_Vertical, F.Cu at (151.5, 57.5)
- added J7: Conn_01x02_Pin, Connector_PinHeader_2.54mm:PinHeader_1x02_P2.54mm_Vertical, F.Cu at (165.5, 57.5)
- added J8: Conn_01x02_Pin, Connector_PinHeader_2.54mm:PinHeader_1x02_P2.54mm_Vertical, F.Cu at (179.5, 57.5)
- added J9: Conn_01x02_Pin, Connector_PinHeader_2.54mm:PinHeader_1x02_P2.54mm_Vertical, F.Cu at (193.5, 57.5)
- added REF**: MountingHole_3.2mm_M3, MountingHole:MountingHole_3.2mm_M3, F.Cu at (104.0, 54.0)
- added REF**: MountingHole_3.2mm_M3, MountingHole:MountingHole_3.2mm_M3, F.Cu at (216.0, 54.0)
- added REF**: MountingHole_3.2mm_M3, MountingHole:MountingHole_3.2mm_M3, F.Cu at (216.0, 136.0)
- added REF**: MountingHole_3.2mm_M3, MountingHole:MountingHole_3.2mm_M3, F.Cu at (104.0, 136.0)
- added VDD: Conn_01x02_Pin, Connector_PinHeader_2.54mm:PinHeader_1x02_P2.54mm_Vertical, F.Cu at (215.9, 78.7)
- moved R23 13.5 mm to (205.7, 78.7)
- moved C14 6.46 mm to (201.5, 83.8)
- moved C15 6.46 mm to (210.8, 83.8)
- moved D6 6.46 mm to (200.7, 78.7), turned to 90 degrees
- moved J4 4.96 mm to (205.6, 62.2)
Connections:
- net Net-(D1-A) renamed CLIP_1
Routing:
- net OUT: track 92.8 -> 102.9 mm
- net TONE_OUT: track 109.3 -> 114.1 mm
- net VDD: track 133.0 -> 137.5 mm
- net Net-(D6-A): track 20.9 -> 16.4 mm
- net CLIP_OUT: track 77.3 -> 80.1 mm
- net Net-(Q1-E): track 17.8 -> 19.0 mm
- net IN: track 60.9 -> 60.1 mm
- net Net-(D5-A): track 7.86 -> 8.42 mm
Other:
- outline, holes or cut-outs redrawn
- board text added: "INPUT"
- board text added: "OUTPUT"
- board text added: "WORKSHOP EDITION"
