File: pcb/bigmuff.kicad_sch (KiCad schematic)
At the start: 66 parts, among them J1 NRJ4HF, J10 Conn_01x02_Pin, J11 Conn_01x02_Pin, J2 NRJ4HF, J3 Conn_01x02_Pin, J4 Barrel_Jack_Switch, J5 Conn_01x02_Pin, J6 Conn_01x02_Pin, J7 Conn_01x02_Pin, J8 Conn_01x02_Pin, J9 Conn_01x02_Pin, Q1 BC549, Q2 BC549, Q3 BC549, Q4 BC549

Commit message: pre-fab update 1
Parts:
- C10: value 4nF -> 3.9nF
Connections:
- net GND: now also R18.1, RV3.1; no longer RV3.3
- net VDD: no longer R18.1
- net at C10.2, R18.2: now also RV2.3; no longer RV2.1
- net at C11.2, R17.2: now also RV2.1; no longer RV2.3
- net at C3.2: now also RV1.3; no longer RV1.1
- net at R6.1: now also RV1.1; no longer RV1.3
- net at C13.2: now also RV3.3; no longer RV3.1

Commit message: pre fab update 2
Parts:
- C1, C6, C8: footprint Capacitor_THT:C_Axial_L5.1mm_D3.1mm_P7.50mm_Horizontal -> Capacitor_THT:C_Rect_L7.2mm_W5.5mm_P5.00mm_FKS2_FKP2_MKS2_MKP2; symbol Device:C_Polarized -> Device:C
- C10, C15, C2, C5, C9: footprint Capacitor_THT:C_Axial_L5.1mm_D3.1mm_P7.50mm_Horizontal -> Capacitor_THT:C_Disc_D5.0mm_W2.5mm_P5.00mm
- C11, C12, C13, C4, C7: footprint Capacitor_THT:C_Axial_L5.1mm_D3.1mm_P7.50mm_Horizontal -> Capacitor_THT:C_Rect_L7.2mm_W2.5mm_P5.00mm_FKS2_FKP2_MKS2_MKP2
- C3: footprint Capacitor_THT:C_Axial_L5.1mm_D3.1mm_P7.50mm_Horizontal -> Capacitor_THT:C_Rect_L7.2mm_W5.5mm_P5.00mm_FKS2_FKP2_MKS2_MKP2
- J1, J2: value NRJ4HF -> NMJ4HFD2; footprint Connector_Audio:Jack_6.35mm_Neutrik_NMJ4HFD3_Horizontal -> Connector_Audio:Jack_6.35mm_Neutrik_NMJ4HFD2_Horizontal; symbol Connector_Audio:NRJ4HF -> Connector_Audio:NMJ4HFD2
- J4: footprint Connector_BarrelJack:BarrelJack_Kycon_KLDX-0202-xC_Horizontal -> bigmuff:BarrelJack_Tayda_A-4118_Horizontal
- RV1, RV2, RV3: footprint Potentiometer_THT:Potentiometer_Alps_RK09L_Single_Vertical -> bigmuff:Potentiometer_Alpha_RD901F-40-00D_RoundLegs
